File: NTC reader/NTC reader.kicad_pcb (KiCad board)
At the start: 2 copper layers, 100.1 x 65 mm, 109 parts, among them IC1 ADG732BSUZ-REEL, IC2 PCA9539RPW_118, J1 43045-1602, J2 43045-1602, J3 Conn_01x05_Pin, J4 Conn_01x03_Pin, J5 Conn_01x03_Pin, J6 43045-1602, J7 43045-1602

Commit message: Removed file
Removed Fixed NTC reader
Routing:
- net /I/O: track 0.00 -> 67.7 mm
- net GND: track 8.93 -> 70.5 mm, vias 3 -> 35
- net /ADG_TEMP_Sense/F_Temp_32: track 25.8 -> 42.5 mm
- net /ADG_TEMP_Sense/F_Temp_31: track 22.5 -> 38.4 mm
- net /ADG_TEMP_Sense/F_Temp_30: track 19.2 -> 34.4 mm
- net /ADG_TEMP_Sense/F_Temp_29: track 15.6 -> 30.0 mm
- net /ADG_TEMP_Sense/F_Temp_16: track 29.5 -> 42.7 mm
- net /ADG_TEMP_Sense/F_Temp_15: track 26.0 -> 38.5 mm
- net /ADG_TEMP_Sense/F_Temp_14: track 22.7 -> 34.4 mm
- net /ADG_TEMP_Sense/F_Temp_28: track 18.5 -> 27.9 mm
- net /ADG_TEMP_Sense/F_Temp_23: track 4.56 -> 13.9 mm
- net /ADG_TEMP_Sense/F_Temp_27: track 16.0 -> 24.7 mm
- net /ADG_TEMP_Sense/F_Temp_26: track 13.4 -> 21.4 mm
- net /ADG_TEMP_Sense/F_Temp_17: track 26.2 -> 33.7 mm
- net /ADG_TEMP_Sense/F_Temp_25: track 10.9 -> 18.1 mm
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Other:
- board size 100.1 x 65 mm -> 100.1 x 59 mm
