File: NTC reader/I-P_Connectors.kicad_sch (KiCad schematic)
At the start: 4 parts, among them J1 43045-1602, J2 43045-1602

Commit message: -
Parts:
- renumbered J2 to J1, J1 to J2, J1 to J6, J2 to J7
Changed lines of the file:
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@@
     (pin "1")
     (instances
-      (project "FIxed NTC reader"
-        (path "/c46dcc17-4871-47d7-b5e1-0a6ae58ced02/d45cf43a-d0e0-470e-aea6-55e44dff3030"
+      (project "Analog Reader(NTC)"
+        (path "/c4414539-6264-4bea-9fce-ce34b2cb5b6b/d45cf43a-d0e0-470e-aea6-55e44dff3030"
           (reference "#PWR014") (unit 1)
         )
       )
+      (project "FIxed NTC reader"
+        (path "/c46dcc17-4871-47d7-b5e1-0a6ae58ced02/d45cf43a-d0e0-470e-aea6-55e44dff3030"
+          (reference "#PWR014") (unit 1)
+        )
+      )
     )
   )
@@
     (pin "1")
     (instances
-      (project "FIxed NTC reader"
-        (path "/c46dcc17-4871-47d7-b5e1-0a6ae58ced02/d45cf43a-d0e0-470e-aea6-55e44dff3030"
+      (project "Analog Reader(NTC)"
+        (path "/c4414539-6264-4bea-9fce-ce34b2cb5b6b/d45cf43a-d0e0-470e-aea6-55e44dff3030"
           (reference "#PWR013") (unit 1)
         )
       )
+      (project "FIxed NTC reader"
+        (path "/c46dcc17-4871-47d7-b5e1-0a6ae58ced02/d45cf43a-d0e0-470e-aea6-55e44dff3030"
+          (reference "#PWR013") (unit 1)
+        )
+      )
     )
   )
   (symbol (lib_id "NTC_Board:43045-1602") (at 88.9 66.04 0) (unit 1)
     (in_bom yes) (on_board yes) (dnp no) (fields_autoplaced)
-    (property "Reference" "J1" (at 100.33 58.42 0)
+    (property "Reference" "J6" (at 100.33 58.42 0)
       (effects (font (size 1.27 1.27)))
     )
@@
     (pin "9")
     (instances
+      (project "Analog Reader(NTC)"
+        (path "/c4414539-6264-4bea-9fce-ce34b2cb5b6b/d45cf43a-d0e0-470e-aea6-55e44dff3030"
+          (reference "J1") (unit 1)
+        )
+      )
       (project "FIxed NTC reader"
         (path "/c46dcc17-4871-47d7-b5e1-0a6ae58ced02"
@@
     (pin "1")
     (instances
-      (project "FIxed NTC reader"
-        (path "/c46dcc17-4871-47d7-b5e1-0a6ae58ced02/d45cf43a-d0e0-470e-aea6-55e44dff3030"
+      (project "Analog Reader(NTC)"
+        (path "/c4414539-6264-4bea-9fce-ce34b2cb5b6b/d45cf43a-d0e0-470e-aea6-55e44dff3030"
           (reference "#PWR011") (unit 1)
         )
       )
+      (project "FIxed NTC reader"
+        (path "/c46dcc17-4871-47d7-b5e1-0a6ae58ced02/d45cf43a-d0e0-470e-aea6-55e44dff3030"
+          (reference "#PWR011") (unit 1)
+        )
+      )
     )
   )
   (symbol (lib_id "NTC_Board:43045-1602") (at 177.8 66.04 0) (unit 1)
     (in_bom yes) (on_board yes) (dnp no) (fields_autoplaced)
-    (property "Reference" "J1" (at 189.23 58.42 0)
+    (property "Reference" "J2" (at 189.23 58.42 0)
       (effects (font (size 1.27 1.27)))
     )
@@
     (pin "9")
     (instances
+      (project "Analog Reader(NTC)"
+        (path "/c4414539-6264-4bea-9fce-ce34b2cb5b6b/d45cf43a-d0e0-470e-aea6-55e44dff3030"
+          (reference "J1") (unit 1)
+        )
+      )
       (project "FIxed NTC reader"
         (path "/c46dcc17-4871-47d7-b5e1-0a6ae58ced02"
@@
     (pin "1")
     (instances
-      (project "FIxed NTC reader"
-        (path "/c46dcc17-4871-47d7-b5e1-0a6ae58ced02/d45cf43a-d0e0-470e-aea6-55e44dff3030"
+      (project "Analog Reader(NTC)"
+        (path "/c4414539-6264-4bea-9fce-ce34b2cb5b6b/d45cf43a-d0e0-470e-aea6-55e44dff3030"
           (reference "#PWR012") (unit 1)
         )
       )
+      (project "FIxed NTC reader"
+        (path "/c46dcc17-4871-47d7-b5e1-0a6ae58ced02/d45cf43a-d0e0-470e-aea6-55e44dff3030"
+          (reference "#PWR012") (unit 1)
+        )
+      )
     )
   )
   (symbol (lib_id "NTC_Board:43045-1602") (at 88.9 114.3 0) (unit 1)
     (in_bom yes) (on_board yes) (dnp no) (fields_autoplaced)
-    (property "Reference" "J2" (at 100.33 106.68 0)
+    (property "Reference" "J7" (at 100.33 106.68 0)
       (effects (font (size 1.27 1.27)))
     )
@@
     (pin "9")
     (instances
+      (project "Analog Reader(NTC)"
+        (path "/c4414539-6264-4bea-9fce-ce34b2cb5b6b/d45cf43a-d0e0-470e-aea6-55e44dff3030"
+          (reference "J2") (unit 1)
+        )
+      )
       (project "FIxed NTC reader"
         (path "/c46dcc17-4871-47d7-b5e1-0a6ae58ced02"
@@
   (symbol (lib_id "NTC_Board:43045-1602") (at 177.8 114.3 0) (unit 1)
     (in_bom yes) (on_board yes) (dnp no) (fields_autoplaced)
-    (property "Reference" "J2" (at 189.23 106.68 0)
+    (property "Reference" "J1" (at 189.23 106.68 0)
       (effects (font (size 1.27 1.27)))
     )
@@
     (pin "9")
     (instances
+      (project "Analog Reader(NTC)"
+        (path "/c4414539-6264-4bea-9fce-ce34b2cb5b6b/d45cf43a-d0e0-470e-aea6-55e44dff3030"
+          (reference "J2") (unit 1)
+        )
+      )
       (project "FIxed NTC reader"
         (path "/c46dcc17-4871-47d7-b5e1-0a6ae58ced02"
